File: Work Package 4/exerc_4_5.brd (EAGLE design)
At the start: 68.6 x 53.3 mm, 6 parts

Commit message: Correctly done 4_5
Parts:
- moved KEYPAD2 63.5 mm to (5.00, 73.6)
- moved R1 12.7 mm to (5.00, 22.8)
- moved R4 12.7 mm to (5.00, 60.9)
- moved U2 12.7 mm to (5.00, 10.1)
- moved R2 12.7 mm to (5.00, 35.5)
- moved R3 12.7 mm to (5.00, 48.2)
Changed lines of the file:
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@@
 </autorouter>
 <elements>
-<element value="" name="KEYPAD2" library="AUTODESK_CIRCUITS_BREADBOARD" package="1X8P-2.54-2.54-11.6-3.0-BLACK-MALE" x="5" y="10.08"></element><element value="" name="U2" library="AUTODESK_CIRCUITS_BREADBOARD" package="ARDUINO_UNO" x="5" y="22.78"></element><element value="1k‎Ω" name="R1" library="AUTODESK_CIRCUITS_BREADBOARD" package="0207/10" x="5" y="35.480000000000004"></element><element value="1k‎Ω" name="R2" library="AUTODESK_CIRCUITS_BREADBOARD" package="0207/10" x="5" y="48.18"></element><element value="1k‎Ω" name="R3" library="AUTODESK_CIRCUITS_BREADBOARD" package="0207/10" x="5" y="60.879999999999995"></element><element value="1k‎Ω" name="R4" library="AUTODESK_CIRCUITS_BREADBOARD" package="0207/10" x="5" y="73.58"></element></elements>
+<element value="" name="U2" library="AUTODESK_CIRCUITS_BREADBOARD" package="ARDUINO_UNO" x="5" y="10.08"></element><element value="1k‎Ω" name="R1" library="AUTODESK_CIRCUITS_BREADBOARD" package="0207/10" x="5" y="22.78"></element><element value="1k‎Ω" name="R2" library="AUTODESK_CIRCUITS_BREADBOARD" package="0207/10" x="5" y="35.480000000000004"></element><element value="1k‎Ω" name="R3" library="AUTODESK_CIRCUITS_BREADBOARD" package="0207/10" x="5" y="48.18"></element><element value="1k‎Ω" name="R4" library="AUTODESK_CIRCUITS_BREADBOARD" package="0207/10" x="5" y="60.879999999999995"></element><element value="" name="KEYPAD2" library="AUTODESK_CIRCUITS_BREADBOARD" package="1X8P-2.54-2.54-11.6-3.0-BLACK-MALE" x="5" y="73.58"></element></elements>
 <signals>
-<signal name="N$1"><contactref element="KEYPAD2" pad="1"></contactref><contactref element="U2" pad="11"></contactref><wire x1="5" y1="18.97" x2="39.036" y2="73.58" width="0" layer="19" extent="1-1"></wire></signal><signal name="N$2"><contactref element="KEYPAD2" pad="2"></contactref><contactref element="U2" pad="10"></contactref><wire x1="5" y1="16.43" x2="41.576" y2="73.58" width="0" layer="19" extent="1-1"></wire></signal><signal name="N$3"><contactref element="KEYPAD2" pad="3"></contactref><contactref element="U2" pad="9"></contactref><wire x1="5" y1="13.89" x2="44.116" y2="73.58" width="0" layer="19" extent="1-1"></wire></signal><signal name="N$4"><contactref element="KEYPAD2" pad="4"></contactref><contactref element="U2" pad="8"></contactref><wire x1="5" y1="11.35" x2="46.656" y2="73.58" width="0" layer="19" extent="1-1"></wire></signal><signal name="N$5"><contactref element="KEYPAD2" pad="5"></contactref><contactref element="U2" pad="7"></contactref><wire x1="5" y1="8.81" x2="50.72" y2="73.58" width="0" layer="19" extent="1-1"></wire><contactref element="R1" pad="2"></contactref><wire x1="50.72" y1="73.58" x2="10.08" y2="35.480000000000004" width="0" layer="19" extent="1-1"></wire></signal><signal name="N$6"><contactref element="KEYPAD2" pad="6"></contactref><contactref element="U2" pad="6"></contactref><wire x1="5" y1="6.27" x2="53.26" y2="73.58" width="0" layer="19" extent="1-1"></wire><contactref element="R2" pad="2"></contactref><wire x1="53.26" y1="73.58" x2="10.08" y2="48.18" width="0" layer="19" extent="1-1"></wire></signal><signal name="N$7"><contactref element="KEYPAD2" pad="7"></contactref><contactref element="U2" pad="5"></contactref><wire x1="5" y1="3.7300000000000004" x2="55.8" y2="73.58" width="0" layer="19" extent="1-1"></wire><contactref element="R3" pad="2"></contactref><wire x1="55.8" y1="73.58" x2="10.08" y2="60.879999999999995" width="0" layer="19" extent="1-1"></wire></signal><signal name="N$8"><contactref element="KEYPAD2" pad="8"></contactref><contactref element="U2" pad="4"></contactref><wire x1="5" y1="1.1899999999999995" x2="58.34" y2="73.58" width="0" layer="19" extent="1-1"></wire><contactref element="R4" pad="2"></contactref><wire x1="58.34" y1="73.58" x2="10.08" y2="73.58" width="0" layer="19" extent="1-1"></wire></signal><signal name="N$9"><contactref element="R4" pad="1"></contactref><contactref element="R3" pad="1"></contactref><wire x1="-0.08000000000000007" y1="73.58" x2="-0.08000000000000007" y2="60.879999999999995" width="0" layer="19" extent="1-1"></wire><contactref element="R2" pad="1"></contactref><wire x1="-0.08000000000000007" y1="60.879999999999995" x2="-0.08000000000000007" y2="48.18" width="0" layer="19" extent="1-1"></wire><contactref element="R1" pad="1"></contactref><wire x1="-0.08000000000000007" y1="48.18" x2="-0.08000000000000007" y2="35.480000000000004" width="0" layer="19" extent="1-1"></wire><contactref element="U2" pad="5V"></contactref><wire x1="-0.08000000000000007" y1="35.480000000000004" x2="43.1" y2="25.32" width="0" layer="19" extent="1-1"></wire></signal></signals>
+<signal name="N$1"><contactref element="U2" pad="11"></contactref><contactref element="KEYPAD2" pad="1"></contactref><wire x1="39.036" y1="60.879999999999995" x2="5" y2="82.47" width="0" layer="19" extent="1-1"></wire></signal><signal name="N$2"><contactref element="U2" pad="10"></contactref><contactref element="KEYPAD2" pad="2"></contactref><wire x1="41.576" y1="60.879999999999995" x2="5" y2="79.92999999999999" width="0" layer="19" extent="1-1"></wire></signal><signal name="N$3"><contactref element="U2" pad="9"></contactref><contactref element="KEYPAD2" pad="3"></contactref><wire x1="44.116" y1="60.879999999999995" x2="5" y2="77.39" width="0" layer="19" extent="1-1"></wire></signal><signal name="N$4"><contactref element="U2" pad="8"></contactref><contactref element="KEYPAD2" pad="4"></contactref><wire x1="46.656" y1="60.879999999999995" x2="5" y2="74.85" width="0" layer="19" extent="1-1"></wire></signal><signal name="N$5"><contactref element="U2" pad="7"></contactref><contactref element="R1" pad="2"></contactref><wire x1="50.72" y1="60.879999999999995" x2="10.08" y2="22.78" width="0" layer="19" extent="1-1"></wire><contactref element="KEYPAD2" pad="5"></contactref><wire x1="10.08" y1="22.78" x2="5" y2="72.31" width="0" layer="19" extent="1-1"></wire></signal><signal name="N$6"><contactref element="U2" pad="6"></contactref><contactref element="R2" pad="2"></contactref><wire x1="53.26" y1="60.879999999999995" x2="10.08" y2="35.480000000000004" width="0" layer="19" extent="1-1"></wire><contactref element="KEYPAD2" pad="6"></contactref><wire x1="10.08" y1="35.480000000000004" x2="5" y2="69.77" width="0" layer="19" extent="1-1"></wire></signal><signal name="N$7"><contactref element="U2" pad="5"></contactref><contactref element="R3" pad="2"></contactref><wire x1="55.8" y1="60.879999999999995" x2="10.08" y2="48.18" width="0" layer="19" extent="1-1"></wire><contactref element="KEYPAD2" pad="7"></contactref><wire x1="10.08" y1="48.18" x2="5" y2="67.23" width="0" layer="19" extent="1-1"></wire></signal><signal name="N$8"><contactref element="U2" pad="4"></contactref><contactref element="R4" pad="2"></contactref><wire x1="58.34" y1="60.879999999999995" x2="10.08" y2="60.879999999999995" width="0" layer="19" extent="1-1"></wire><contactref element="KEYPAD2" pad="8"></contactref><wire x1="10.08" y1="60.879999999999995" x2="5" y2="64.69" width="0" layer="19" extent="1-1"></wire></signal><signal name="N$9"><contactref element="R4" pad="1"></contactref><contactref element="R3" pad="1"></contactref><wire x1="-0.08000000000000007" y1="60.879999999999995" x2="-0.08000000000000007" y2="48.18" width="0" layer="19" extent="1-1"></wire><contactref element="R2" pad="1"></contactref><wire x1="-0.08000000000000007" y1="48.18" x2="-0.08000000000000007" y2="35.480000000000004" width="0" layer="19" extent="1-1"></wire><contactref element="R1" pad="1"></contactref><wire x1="-0.08000000000000007" y1="35.480000000000004" x2="-0.08000000000000007" y2="22.78" width="0" layer="19" extent="1-1"></wire><contactref element="U2" pad="5V"></contactref><wire x1="-0.08000000000000007" y1="22.78" x2="43.1" y2="12.620000000000001" width="0" layer="19" extent="1-1"></wire></signal></signals>
 </board>
 </drawing>
